Commit message: changed the gravel error, added gripper_tool_frame and base collision box + colors

File: robots/hsrb4s.obj.urdf (robot description, URDF)
Before this commit: robot hsrb, 45 links, 44 joints
Links:
- added link gripper_tool_frame
Joints:
- added joint gripper_tool_joint: type fixed, parent hand_palm_link, child gripper_tool_frame, origin xyz=0.012 0.0 0.075 rpy=0.0 0.0 -80.14159265359
